Commit message: Created world

File: description/robot.urdf.xacro (robot description, xacro)
@@ -2,3 +2,4 @@
 <robot xmlns:xacro="http://www.ros.org/wiki/xacro"  name="robot">
    <xacro:include filename="robot_core.xacro" />
+   <xacro:include filename="gazebo_control.xacro"/>
 </robot>

File: description/robot_core.xacro (robot description, xacro)
@@ -2,20 +2,20 @@
 <robot xmlns:xacro="http://www.ros.org/wiki/xacro" >
     <xacro:include filename="inertial_macros.xacro"/>
-    <material name="white" >
+    <material name="white">
         <color rgba="1 1 1 1" />
     </material>
-    <material name="orange" >
-        <color rgba="1 0.3 0.1 1" />
+    <material name="orange">
+        <color rgba="1 0.3 0.1 1"/>
     </material>
-    <material name="blue" >
-        <color rgba="0.2 0.2 1 1" />
+    <material name="blue">
+        <color rgba="0.2 0.2 1 1"/>
     </material>
-    <material name="black" >
-        <color rgba="0 0 0 1" />
+    <material name="black">
+        <color rgba="0 0 0 1"/>
     </material>
     <!-- BASE LINK -->
     <link name="base_link">
     </link>
-    <!-- CHASSIS LINK-->
+    <!-- CHASSIS LINK -->
     <joint name="chassis_joint" type="fixed">
         <parent link="base_link"/>
@@ -38,12 +38,15 @@
         </collision>
         <xacro:inertial_box mass="0.5" x="0.3" y="0.3" z="0.15">
-            <origin xyz="0.15 0 0.75" rpy="0 0 0"/>
+            <origin xyz="0.15 0 0.075" rpy="0 0 0"/>
         </xacro:inertial_box>
     </link>
-    <!-- LEFT WHEEL LINK-->
+    <gazebo reference="chassis">
+        <material>Gazebo/White</material>
+    </gazebo>
+    <!-- LEFT WHEEL LINK -->
     <joint name="left_wheel_joint" type="continuous">
         <parent link="base_link"/>
         <child link="left_wheel"/>
-        <origin xyz="0 0.175 0" rpy="-${pi/2} 0 0"/>
+        <origin xyz="0 0.175 0" rpy="-${pi/2} 0 0" />
         <axis xyz="0 0 1"/>
     </joint>
@@ -64,9 +67,12 @@
         </xacro:inertial_cylinder>
     </link>
-    <!-- RIGHT WHEEL LINK-->
+    <gazebo reference="left_wheel">
+        <material>Gazebo/Blue</material>
+    </gazebo>
+    <!-- RIGHT WHEEL LINK -->
     <joint name="right_wheel_joint" type="continuous">
         <parent link="base_link"/>
         <child link="right_wheel"/>
-        <origin xyz="0 -0.175 0" rpy="${pi/2} 0 0"/>
+        <origin xyz="0 -0.175 0" rpy="${pi/2} 0 0" />
         <axis xyz="0 0 -1"/>
     </joint>
@@ -87,6 +93,9 @@
         </xacro:inertial_cylinder>
     </link>
-    <!-- CASTER WHEE LINK-->
-    <joint name="caster_wheel_link" type="fixed">
+    <gazebo reference="right_wheel">
+        <material>Gazebo/Blue</material>
+    </gazebo>
+    <!-- CASTER WHEEL LINK -->
+    <joint name="caster_wheel_joint" type="fixed">
         <parent link="chassis"/>
         <child link="caster_wheel"/>
@@ -100,5 +109,5 @@
             <material name="black"/>
         </visual>
-         <collision>
+        <collision>
             <geometry>
                 <sphere radius="0.05"/>
@@ -109,3 +118,8 @@
         </xacro:inertial_sphere>
     </link>
+    <gazebo reference="caster_wheel">
+        <material>Gazebo/Black</material>
+        <mu1 value="0.001"/>
+        <mu2 value="0.001"/>
+    </gazebo>
 </robot>
